File: Esquematico_y_PCB/Diseño_de_FISICA_v16.brd (EAGLE design)
At the start: 100 x 80 mm, 39 parts, among them IC1 2133-DRV8825, IC2 2133-DRV8825, IC3 2133-DRV8825, J2 3A/250V

Commit message: Acualización PCB y SCH
Parts:
- removed GPIO_DIG2: PINHD-1X8, Connector:1X08
- removed J2: 3A/250V, Connector:B2B-XH-A
- removed JP1, JP2, JP3: (no value), adafruit:1X1-BIGPOGO
- removed LED7: (no value), led:LED3MM
- removed MOTOR_4: PINHD-1X4, Connector:1X04
- removed R7: (no value), Resistor:RESC2012X65
- added DIG: PINHD-1X4, Connector:1X04
- added J1, VIN, VOUT: 1X2-3.5MM, adafruit:1X2-3.5MM
- added S1: (no value), switch:M9040P
- added UART_0: PINHD-1X3, Connector:1X03
- GPIO_DIG: value PINHD-1X8 -> (none); device Connector:1X08 -> pinhead:2X10
- R2, R3: device Resistor:RESC2012X65 -> rcl:0309/10
- moved R2 33.6 mm to (35.6, 69.8), flipped to the top, turned to 270 degrees
- moved LED2 31.9 mm to (40.6, 66.0), turned to 90 degrees
- moved R4 17.1 mm to (17.8, 55.9)
- moved SERV_1 16.6 mm to (45.7, 69.8), turned to 90 degrees
- moved LED4 16.3 mm to (21.6, 55.9)
- moved R5 16.2 mm to (17.8, 49.5)
- moved R3 16.2 mm to (17.8, 69.8), flipped to the top, turned to 270 degrees
- moved LED5 15.3 mm to (21.6, 49.5)
- moved R6 15.3 mm to (17.8, 43.2)
- moved MODULO_ETHERNET 15.3 mm to (53.3, 19.1)
- moved LED6 14.4 mm to (21.6, 43.2)
- moved SERV_2 14.0 mm to (27.9, 69.8), turned to 270 degrees
- moved LED3 13.7 mm to (22.9, 66.0), turned to 90 degrees
- moved UART_2 10.8 mm to (71.1, 67.3)
- moved RELAYS 9.25 mm to (95.2, 53.3)
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Connections:
- removed net AREF: ARDUINOMEGA2560.AREF, MOTOR_4.4
- removed net GND1: IC1.9, IC2.9, IC3.9
- removed net LED_AUX: ARDUINOMEGA2560.11, LED7.A
- removed net N$37: LED7.K, R7.2
- removed net RST: ARDUINOMEGA2560.RESET, MOTOR_4.3
- removed net VCC: J2.1, JP1.P$1, SERV_1.2, SERV_2.2
- new net GND_MOT: IC1.15, IC2.15, IC3.15, J1.1
- new net N$1: S1.2, VIN.2
- new net N$2: S1.3, VOUT.1
- new net N$3: VIN.1, VOUT.2
- net CLK: now also GPIO_DIG.18; no longer MODULO_ETHERNET.CLK
- net D20: now also DIG.1; no longer GPIO_DIG2.7
- net D21: now also DIG.2; no longer GPIO_DIG2.8
- net D40: now also GPIO_DIG.9; no longer GPIO_DIG2.1
- net D41: now also GPIO_DIG.10; no longer GPIO_DIG2.2
- net D42: now also GPIO_DIG.11; no longer GPIO_DIG2.3
- net D43: now also GPIO_DIG.12; no longer GPIO_DIG2.4
- net D44: now also GPIO_DIG.13; no longer GPIO_DIG2.5
- net D45: now also GPIO_DIG.14; no longer GPIO_DIG2.6
- net GND: now also DIG.3, DIG.4, GPIO_DIG.19, GPIO_DIG.20, IC1.1, IC1.9, IC2.1, IC2.9, IC3.1, IC3.9, UART_0.3; no longer IC1.15, IC2.15, IC3.15, J2.2, JP3.P$1, R7.1
- net LED_SERV_1: now also ARDUINOMEGA2560.7; no longer ARDUINOMEGA2560.12
- net NT: now also GPIO_DIG.15; no longer MODULO_ETHERNET.NT
- net PWM_SERV_2: now also ARDUINOMEGA2560.12; no longer ARDUINOMEGA2560.7
- net RST_1: now also GPIO_DIG.17; no longer MODULO_ETHERNET.RST
- net RX: now also UART_0.2; no longer MOTOR_4.2
- net TX: now also UART_0.1; no longer MOTOR_4.1
- net VCC_5: now also SERV_1.2, SERV_2.2; no longer JP2.P$1
- net VCC_MOT: now also J1.2
- net WOL: now also GPIO_DIG.16; no longer MODULO_ETHERNET.WOL
Routing:
- net GND: track 0.00 -> 573.6 mm
- net VCC_5: track 0.00 -> 138.2 mm, vias 0 -> 2
- net GND_MOT: track 0.00 -> 91.0 mm
- net VCC_MOT: track 0.00 -> 88.2 mm, vias 0 -> 4
- net VCC_3_3: track 0.00 -> 50.1 mm
- net DIR_1: track 0.00 -> 48.4 mm
- net STEP_1: track 0.00 -> 45.8 mm
- net N$3: track 0.00 -> 33.5 mm
- net CLK: track 32.6 -> 3.81 mm
- net DIR_2: track 0.00 -> 27.0 mm
- net LED_MOT_1: track 0.00 -> 24.8 mm
- net STEP_2: track 0.00 -> 24.5 mm
- net SO: track 20.2 -> 43.6 mm
- net WOL: track 26.6 -> 3.81 mm
- net CS: track 20.8 -> 43.0 mm
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- added copper zone on layer 16, net GND
Other:
- board size 100 x 80 mm -> 100 x 77.5 mm

Commit message: cambios PCB
Parts:
- removed DIG: PINHD-1X4, Connector:1X04
- removed UART_2: PINHD-1X3, Connector:1X03
- added D1: 1N4004, adafruit:DO41-10
- added K1: 351, relay:351
- added R7: (no value), Resistor:RESC2012X65
- added SW_M1, SW_M2, SW_M3: (no value), pinhead:2X02
- added VIN1, VIN2: 1X2-3.5MM, adafruit:1X2-3.5MM
- moved ANALOG_1 2.54 mm to (52.2, 5.08)
- moved 3-3VCC 2.54 mm to (19.1, 5.08)
- moved 5_VCC 2.54 mm to (27.9, 5.08)
- moved ANALOG_2 2.54 mm to (74.9, 5.08)
- moved GND 2.54 mm to (36.8, 5.08)
- moved MODULO_ETHERNET 2.04 mm to (53.2, 17.0)
- moved R5 0.25 mm to (17.5, 49.5)
- moved R6 0.25 mm to (17.5, 43.2)
- moved R4 0.13 mm to (17.7, 55.9)
Connections:
- removed net D20: ARDUINOMEGA2560.20, DIG.1
- removed net D21: ARDUINOMEGA2560.21, DIG.2
- removed net GND_MOT: IC1.15, IC2.15, IC3.15, J1.1
- removed net RX_1: ARDUINOMEGA2560.19, UART_2.3
- removed net RX_2: ARDUINOMEGA2560.17, UART_2.1
- removed net TX_1: ARDUINOMEGA2560.18, UART_2.2
- removed net TX_2: ARDUINOMEGA2560.16, UART_1.3
- new net N$10: D1.A, K1.16, R7.2
- new net N$11: K1.S1, VIN1.1
- new net N$12: K1.S2, VIN2.1
- new net N$4: IC1.10
- new net N$5: IC2.10
- new net N$6: IC3.10
- new net SW_M1_FIN: ARDUINOMEGA2560.17, SW_M1.3
- new net SW_M1_INIT: ARDUINOMEGA2560.16, SW_M1.1
- new net SW_M2_FIN: ARDUINOMEGA2560.19, SW_M2.3
- new net SW_M2_INIT: ARDUINOMEGA2560.18, SW_M2.1
- new net SW_M3_FIN: ARDUINOMEGA2560.21, SW_M3.3
- new net SW_M3_INIT: ARDUINOMEGA2560.20, SW_M3.1
- new net VCC_SERVO: K1.P1, SERV_1.2, SERV_2.2
- net GND: now also IC1.15, IC2.15, IC3.15, J1.1, R7.1, SW_M1.2, SW_M1.4, SW_M2.2, SW_M2.4, SW_M3.2, SW_M3.4, UART_1.3, VIN1.2, VIN2.2; no longer ARDUINOMEGA2560.GND@4, ARDUINOMEGA2560.GND@5, DIG.3, DIG.4
- net N$2: now also D1.C, K1.1
- net VCC_5: now also ARDUINOMEGA2560.GND@4, ARDUINOMEGA2560.GND@5; no longer SERV_1.2, SERV_2.2
- net VCC_MOT: now also K1.P2
Routing:
- net GND: track 573.6 -> 682.0 mm, vias 0 -> 2
- net GND_MOT: track 91.0 -> 0.00 mm
- net N$3: track 33.5 -> 0.00 mm
- net VCC_5: track 138.2 -> 107.7 mm
- net SO: track 43.6 -> 57.2 mm
- net D21: track 9.94 -> 0.00 mm
- net D20: track 9.20 -> 0.00 mm
- net TX_2: track 6.35 -> 0.00 mm
- net TX_1: track 6.35 -> 0.00 mm
- net RX_2: track 6.35 -> 0.00 mm
- net RX_1: track 6.35 -> 0.00 mm
- net SI: track 37.4 -> 42.9 mm
- net CS: track 43.0 -> 37.7 mm
- net N$2: track 4.93 -> 0.00 mm
- net A7: track 5.08 -> 7.67 mm
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Other:
- board size 100 x 77.5 mm -> 100 x 78.7 mm

Commit message: modificación esquematico
Parts:
- removed D1: 1N4004, adafruit:DO41-10
- removed K1: 351, relay:351
- removed R7: (no value), Resistor:RESC2012X65
- removed S1: (no value), switch:M9040P
- removed VIN1, VIN2, VOUT: 1X2-3.5MM, adafruit:1X2-3.5MM
- added J2, J3: 1X2-3.5MM, adafruit:1X2-3.5MM
Connections:
- net CLK renamed D49
- net NT renamed D46
- net RST_1 renamed D48
- net WOL renamed D47
- removed net N$1: S1.2, VIN.2
- removed net N$10: D1.A, K1.16, R7.2
- removed net N$11: K1.S1, VIN1.1
- removed net N$12: K1.S2, VIN2.1
- removed net N$2: D1.C, K1.1, S1.3, VOUT.1
- removed net N$3: VIN.1, VOUT.2
- removed net N$4: IC1.10
- removed net N$5: IC2.10
- removed net N$6: IC3.10
- new net FOCO_PIN: ARDUINOMEGA2560.31
- new net LED_AUX: ARDUINOMEGA2560.11
- new net M1_ENABLE: ARDUINOMEGA2560.28, IC1.1
- new net M2_ENABLE: ARDUINOMEGA2560.29, IC2.1
- new net M3_ENABLE: ARDUINOMEGA2560.30, IC3.1
- net D28: no longer ARDUINOMEGA2560.28
- net D29: no longer ARDUINOMEGA2560.29
- net D30: no longer ARDUINOMEGA2560.30
- net D31: no longer ARDUINOMEGA2560.31
- net GND: now also J2.1, J3.1, VIN.1; no longer IC1.1, IC2.1, IC3.1, R7.1, VIN1.2, VIN2.2
- net VCC_5: now also IC1.10, IC2.10, IC3.10, VIN.2
- net VCC_MOT: now also J2.2; no longer K1.P2
- net VCC_SERVO: now also J3.2; no longer K1.P1
Routing:
- net GND: track 682.0 -> 665.0 mm
- net N$1: track 15.4 -> 0.00 mm
- net D31: track 6.88 -> 1.80 mm
- net D30: track 10.5 -> 8.67 mm
- net D28: track 13.0 -> 11.2 mm
- net D29: track 8.82 -> 7.04 mm

Commit message: Modif PCB
Parts:
- removed J2, VIN: 1X2-3.5MM, adafruit:1X2-3.5MM
- added D1: 1N4004, diode:DO41-10
- added Q1: BC817-25SMD, transistor-npn:SOT23-BEC
- added R7: (no value), Resistor:RESC2012X65
- added U$1: RELAY, RELAY:RELAY
- added VIN1: 1X2-3.5MM, adafruit:1X2-3.5MM
- moved SW_M3 131.1 mm to (81.3, 72.4)
- moved SW_M2 119.4 mm to (76.2, 72.4)
- moved J3 109.6 mm to (8.89, 45.7), turned to 90 degrees
- moved SW_M1 108.3 mm to (71.1, 72.4)
- moved UART_0 4.58 mm to (52.1, 69.8)
- moved UART_1 4.58 mm to (59.7, 69.8)
Connections:
- removed net LED_AUX: ARDUINOMEGA2560.11
- new net N$1: U$1.COM_CPEN, VIN1.1
- new net N$2: D1.A, Q1.C, U$1.P$2
- new net N$3: U$1.COM-CLOSE, VIN1.2
- new net N$4: Q1.B, R7.1
- net FOCO_PIN: now also R7.2
- net GND: now also Q1.E; no longer J2.1, VIN.1
- net VCC_5: now also D1.C, U$1.P$1; no longer VIN.2
- net VCC_MOT: no longer J2.2
Routing:
- net GND: track 665.0 -> 581.9 mm
- net VCC_5: track 107.7 -> 39.1 mm
- net VCC_3_3: track 52.6 -> 17.6 mm
- net VCC_MOT: track 88.2 -> 75.1 mm
- net TX_3: track 6.35 -> 10.5 mm
- net TX: track 6.35 -> 10.5 mm
- net RX_3: track 6.35 -> 10.5 mm
- net RX: track 6.35 -> 10.5 mm
- net CS: track 37.7 -> 38.7 mm

Commit message: PCB Corregidas
Parts:
- removed RELAYS: PINHD-1X4, Connector:1X04
- R2, R3: device rcl:0309/10 -> Resistor:RESC2012X65
- moved LED4 45.7 mm to (67.3, 57.1)
- moved R4 44.5 mm to (62.1, 57.1)
- moved LED5 25.3 mm to (45.7, 57.1)
- moved R5 24.9 mm to (41.3, 57.1)
- moved MOTOR_1 24.4 mm to (32.8, 57.3)
- moved MOTOR_2 24.2 mm to (54.6, 57.1)
- moved MOTOR_3 24.2 mm to (76.2, 57.1)
- moved R7 22.9 mm to (61.0, 30.5), flipped to the bottom, turned to 270 degrees
- moved J3 21.6 mm to (7.62, 67.3)
- moved J1 20.4 mm to (7.62, 54.6)
- moved D1 18.1 mm to (72.4, 35.6), turned to 180 degrees
- moved LED6 14.2 mm to (24.1, 57.1)
- moved R6 14.2 mm to (20.1, 57.1)
- moved Q1 10.2 mm to (62.2, 34.3), flipped to the bottom, turned to 90 degrees
- moved R3 10.2 mm to (26.7, 64.8), flipped to the bottom
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Connections:
- removed net D2: ARDUINOMEGA2560.2
- removed net D28: RELAYS.1
- removed net D29: RELAYS.2
- removed net D3: ARDUINOMEGA2560.3
- removed net D30: RELAYS.3
- removed net D4: ARDUINOMEGA2560.4
- removed net D5: ARDUINOMEGA2560.5
- removed net N$21: LED2.K, R2.2
- removed net N$22: LED3.K, R3.2
- new net N$5: LED2.A, R2.1
- new net N$6: LED3.A, R3.1
- net D31: now also ARDUINOMEGA2560.31; no longer RELAYS.4
- net D32: no longer ARDUINOMEGA2560.32
- net D33: no longer ARDUINOMEGA2560.33
- net D34: no longer ARDUINOMEGA2560.34
- net D35: no longer ARDUINOMEGA2560.35
- net D36: no longer ARDUINOMEGA2560.36
- net D37: no longer ARDUINOMEGA2560.37
- net D42: no longer ARDUINOMEGA2560.42
- net D43: no longer ARDUINOMEGA2560.43
- net D44: no longer ARDUINOMEGA2560.44
- net D45: no longer ARDUINOMEGA2560.45
- net D46: no longer ARDUINOMEGA2560.46
- net D47: no longer ARDUINOMEGA2560.47
- net D48: no longer ARDUINOMEGA2560.48
- net DIR_1: now also ARDUINOMEGA2560.30; no longer ARDUINOMEGA2560.23
- net DIR_2: now also ARDUINOMEGA2560.34; no longer ARDUINOMEGA2560.25
- net DIR_3: now also ARDUINOMEGA2560.37; no longer ARDUINOMEGA2560.27
- net FOCO_PIN: now also ARDUINOMEGA2560.48; no longer ARDUINOMEGA2560.31
- net GND: now also LED2.K, LED3.K; no longer R2.1, R3.1
- net LED_MOT_1: no longer ARDUINOMEGA2560.8
- net LED_MOT_2: now also ARDUINOMEGA2560.3; no longer ARDUINOMEGA2560.9
- net LED_MOT_3: now also ARDUINOMEGA2560.2; no longer ARDUINOMEGA2560.10
- net LED_SERV_1: now also ARDUINOMEGA2560.5, R2.2; no longer ARDUINOMEGA2560.7, LED2.A
- net LED_SERV_2: now also ARDUINOMEGA2560.11, R3.2; no longer ARDUINOMEGA2560.13, LED3.A
- net M2_ENABLE: now also ARDUINOMEGA2560.32; no longer ARDUINOMEGA2560.29
- net M3_ENABLE: now also ARDUINOMEGA2560.35; no longer ARDUINOMEGA2560.30
- net N$1: now also VIN1.2; no longer VIN1.1
- net N$3: now also U$1.COM, VIN1.1; no longer U$1.COM-CLOSE, VIN1.2
- net PWM_SERV_1: now also ARDUINOMEGA2560.4; no longer ARDUINOMEGA2560.6
- net PWM_SERV_2: now also ARDUINOMEGA2560.10; no longer ARDUINOMEGA2560.12
- net RX: now also UART_0.1; no longer UART_0.2
- net RX_3: now also UART_1.1; no longer UART_1.2
- net STEP_1: now also ARDUINOMEGA2560.29; no longer ARDUINOMEGA2560.22
- net STEP_2: now also ARDUINOMEGA2560.33; no longer ARDUINOMEGA2560.24
- net STEP_3: now also ARDUINOMEGA2560.36; no longer ARDUINOMEGA2560.26
- net TX: now also UART_0.2; no longer UART_0.1
- net TX_3: now also UART_1.2; no longer UART_1.1
Routing:
- net GND: track 581.9 -> 299.6 mm
- net VCC_5: track 39.1 -> 163.3 mm, vias 2 -> 3
- net M1_ENABLE: track 0.00 -> 73.0 mm, vias 0 -> 2
- net VCC_SERVO: track 0.00 -> 48.7 mm, vias 0 -> 3
- net M2_ENABLE: track 0.00 -> 48.6 mm
- net N$3: track 0.00 -> 39.4 mm, vias 0 -> 2
- net VCC_3_3: track 17.6 -> 55.3 mm, vias 0 -> 2
- net FOCO_PIN: track 0.00 -> 27.1 mm
- net M3_ENABLE: track 0.00 -> 26.3 mm
- net LED_MOT_1: track 24.8 -> 3.57 mm
- net SO: track 57.2 -> 39.3 mm
- net N$1: track 0.00 -> 16.5 mm
- net MOT2_A2: track 21.1 -> 5.93 mm
- net MOT3_A2: track 20.9 -> 5.93 mm
- net MOT1_A2: track 20.9 -> 5.95 mm
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- removed copper zone on layer 16, net GND

Commit message: Diseño PCB full
Parts:
- removed GPIO_DIG: (no value), pinhead:2X10
- removed J1, J3, VIN1: 1X2-3.5MM, adafruit:1X2-3.5MM
- added JP1, JP2, JP3: (no value), adafruit:2X04
- added R8: (no value), Resistor:RESC2012X65
- added RESET: (no value), switch-omron:B3F-10XX
- added X1, X2, X3: (no value), con-ptr500:AK300/2
- moved R1 10.5 mm to (8.89, 1.27), turned to 90 degrees
- moved LED1 6.48 mm to (12.7, 1.27), turned to 180 degrees
- moved MODULO_ETHERNET 4.80 mm to (55.8, 17.9)
- moved 3-3VCC 3.81 mm to (19.1, 1.27)
- moved 5_VCC 3.81 mm to (27.9, 1.27)
- moved ANALOG_1 3.81 mm to (52.2, 1.27)
- moved ANALOG_2 3.81 mm to (74.9, 1.27)
- moved GND 3.81 mm to (36.8, 1.27)
Connections:
- removed net D32: GPIO_DIG.1
- removed net D33: GPIO_DIG.2
- removed net D34: GPIO_DIG.3
- removed net D35: GPIO_DIG.4
- removed net D36: GPIO_DIG.5
- removed net D37: GPIO_DIG.6
- removed net D48: GPIO_DIG.17
- new net D22: ARDUINOMEGA2560.22, JP3.4
- new net D23: ARDUINOMEGA2560.23, JP3.3
- new net D24: ARDUINOMEGA2560.24, JP3.6
- new net D25: ARDUINOMEGA2560.25, JP3.5
- new net D26: ARDUINOMEGA2560.26, JP3.8
- new net D27: ARDUINOMEGA2560.27, JP3.7
- new net RESET: ARDUINOMEGA2560.RESET, R8.2, RESET.3
- net D38: now also JP1.4; no longer GPIO_DIG.7
- net D39: now also JP1.3; no longer GPIO_DIG.8
- net D40: now also JP1.6; no longer GPIO_DIG.9
- net D41: now also JP1.5; no longer GPIO_DIG.10
- net D42: now also ARDUINOMEGA2560.42, JP1.8; no longer GPIO_DIG.11
- net D43: now also ARDUINOMEGA2560.43, JP1.7; no longer GPIO_DIG.12
- net D44: now also ARDUINOMEGA2560.44, JP2.2; no longer GPIO_DIG.13
- net D45: now also ARDUINOMEGA2560.45, JP2.1; no longer GPIO_DIG.14
- net D46: now also ARDUINOMEGA2560.46, JP2.4; no longer GPIO_DIG.15
- net D47: now also ARDUINOMEGA2560.47, JP2.3; no longer GPIO_DIG.16
- net D49: now also JP2.5; no longer GPIO_DIG.18
- net GND: now also JP1.1, JP1.2, JP2.6, JP2.7, JP2.8, RESET.1, X1.1, X2.1; no longer GPIO_DIG.19, GPIO_DIG.20, J1.1, J3.1
- net N$1: now also X3.2; no longer VIN1.2
- net N$3: now also X3.1; no longer VIN1.1
- net VCC_5: now also JP3.1, JP3.2, R8.1
- net VCC_MOT: now also X2.2; no longer J1.2
- net VCC_SERVO: now also X1.2; no longer J3.2
Routing:
- net GND: track 299.6 -> 529.5 mm, vias 2 -> 0
- net RESET: track 0.00 -> 42.9 mm
- net VCC_5: track 163.3 -> 186.8 mm, vias 3 -> 5
- net D42: track 0.00 -> 11.2 mm
- net D40: track 0.00 -> 11.2 mm
- net D38: track 0.00 -> 11.2 mm
- net D26: track 0.00 -> 11.2 mm
- net D24: track 0.00 -> 11.2 mm
- net D22: track 0.00 -> 11.2 mm
- net D46: track 0.00 -> 11.2 mm
- net D44: track 0.00 -> 11.2 mm
- net VCC_3_3: track 55.3 -> 61.5 mm
- net N$3: track 39.4 -> 45.5 mm
- net D49: track 0.00 -> 5.08 mm
- net D47: track 0.00 -> 5.08 mm
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- added copper zone on layer 1, net GND
- added copper zone on layer 16, net GND
Other:
- board size 100 x 78.7 mm -> 100.1 x 79 mm

Commit message: Correcciones PCB
Parts:
- renumbered JP1 to DAUX_1, JP2 to DAUX2, JP3 to DAUX_3, LED1 to LED.ON, LED2 to LS_1, LED3 to LS_2, LED4 to LM_3, LED5 to LM_2, LED6 to LM_1, X1 to +6V, X2 to +12V, X3 to FOCO
Connections:
- net LED_MOT_1: now also ARDUINOMEGA2560.12
Routing:
- net LED_MOT_1: track 3.57 -> 4.63 mm
