File: Esquematico_y_PCB/Diseño_de_FISICA_v16.sch (EAGLE design)
At the start: 37 parts, among them IC1 2133-DRV8825, IC2 2133-DRV8825, IC3 2133-DRV8825, J1 1X2-3.5MM

Commit message: cambios PCB
Parts:
- removed DIG: PINHD-1X4, Connector:PINHD-1X4
- removed UART_2: PINHD-1X3, Connector:PINHD-1X3
- added D1: 1N4004, adafruit:1N4004
- added K1: 351, relay:351
- added R7: (no value), Resistor:R_CHIP-0805(2012-METRIC)
- added SW_M1, SW_M2, SW_M3: (no value), pinhead:PINHD-2X2
- added VIN1, VIN2: 1X2-3.5MM, adafruit:1X2-3.5MM
Connections:
- removed net D20: ARDUINOMEGA2560.20, DIG.1
- removed net D21: ARDUINOMEGA2560.21, DIG.2
- removed net GND_MOT: IC1.GND2, IC2.GND2, IC3.GND2, J1.1
- removed net RX_1: ARDUINOMEGA2560.19, UART_2.3
- removed net RX_2: ARDUINOMEGA2560.17, UART_2.1
- removed net TX_1: ARDUINOMEGA2560.18, UART_2.2
- removed net TX_2: ARDUINOMEGA2560.16, UART_1.3
- new net N$10: D1.A, K11.2, R7.2
- new net N$11: K12.S, VIN1.1
- new net N$12: K13.S, VIN2.1
- new net N$4: IC1.!FLT
- new net N$5: IC2.!FLT
- new net N$6: IC3.!FLT
- new net SW_M1_FIN: ARDUINOMEGA2560.17, SW_M1.3
- new net SW_M1_INIT: ARDUINOMEGA2560.16, SW_M1.1
- new net SW_M2_FIN: ARDUINOMEGA2560.19, SW_M2.3
- new net SW_M2_INIT: ARDUINOMEGA2560.18, SW_M2.1
- new net SW_M3_FIN: ARDUINOMEGA2560.21, SW_M3.3
- new net SW_M3_INIT: ARDUINOMEGA2560.20, SW_M3.1
- new net VCC_SERVO: K12.P, SERV_1.2, SERV_2.2
- net GND: now also IC1.GND2, IC2.GND2, IC3.GND2, J1.1, R7.1, SW_M1.2, SW_M1.4, SW_M2.2, SW_M2.4, SW_M3.2, SW_M3.4, UART_1.3, VIN1.2, VIN2.2; no longer ARDUINOMEGA2560.GND@4, ARDUINOMEGA2560.GND@5, DIG.3, DIG.4
- net N$2: now also D1.C, K11.1
- net VCC_5: now also ARDUINOMEGA2560.GND@4, ARDUINOMEGA2560.GND@5; no longer SERV_1.2, SERV_2.2
- net VCC_MOT: now also K13.P
Other:
- moved on the sheet: S1, UART_0

Commit message: modificación esquematico
Parts:
- removed D1: 1N4004, adafruit:1N4004
- removed K1: 351, relay:351
- removed R7: (no value), Resistor:R_CHIP-0805(2012-METRIC)
- removed S1: (no value), switch:M9040P
- removed VIN1, VIN2, VOUT: 1X2-3.5MM, adafruit:1X2-3.5MM
- added J2, J3: 1X2-3.5MM, adafruit:1X2-3.5MM
Connections:
- net CLK renamed D49
- net NT renamed D46
- net RST_1 renamed D48
- net WOL renamed D47
- removed net N$1: S1.P, VIN.2
- removed net N$10: D1.A, K11.2, R7.2
- removed net N$11: K12.S, VIN1.1
- removed net N$12: K13.S, VIN2.1
- removed net N$2: D1.C, K11.1, S1.S, VOUT.1
- removed net N$3: VIN.1, VOUT.2
- removed net N$4: IC1.!FLT
- removed net N$5: IC2.!FLT
- removed net N$6: IC3.!FLT
- new net FOCO_PIN: ARDUINOMEGA2560.31
- new net LED_AUX: ARDUINOMEGA2560.11
- new net M1_ENABLE: ARDUINOMEGA2560.28, IC1.!EN
- new net M2_ENABLE: ARDUINOMEGA2560.29, IC2.!EN
- new net M3_ENABLE: ARDUINOMEGA2560.30, IC3.!EN
- net D28: no longer ARDUINOMEGA2560.28
- net D29: no longer ARDUINOMEGA2560.29
- net D30: no longer ARDUINOMEGA2560.30
- net D31: no longer ARDUINOMEGA2560.31
- net GND: now also J2.1, J3.1, VIN.1; no longer IC1.!EN, IC2.!EN, IC3.!EN, R7.1, VIN1.2, VIN2.2
- net VCC_5: now also IC1.!FLT, IC2.!FLT, IC3.!FLT, VIN.2
- net VCC_MOT: now also J2.2; no longer K13.P
- net VCC_SERVO: now also J3.2; no longer K12.P

Commit message: Modif PCB
Parts:
- removed J2, VIN: 1X2-3.5MM, adafruit:1X2-3.5MM
- added D1: 1N4004, diode:1N4004
- added Q1: BC817-25SMD, transistor-npn:BC817-25SMD
- added R7: (no value), Resistor:R_CHIP-0805(2012-METRIC)
- added U$1: RELAY, RELAY:RELAY
- added VIN1: 1X2-3.5MM, adafruit:1X2-3.5MM
Connections:
- removed net LED_AUX: ARDUINOMEGA2560.11
- new net N$1: U$1.COM-OPEN, VIN1.1
- new net N$2: D1.A, Q1.C, U$1.GND
- new net N$3: U$1.COM-CLOSE, VIN1.2
- new net N$4: Q1.B, R7.1
- net FOCO_PIN: now also R7.2
- net GND: now also Q1.E; no longer J2.1, VIN.1
- net VCC_5: now also D1.C, U$1.IN; no longer VIN.2
- net VCC_MOT: no longer J2.2
Changed lines of the file:
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@@
 <part name="LED5" library="led" library_urn="urn:adsk.eagle:library:259" deviceset="LED" device="3MM" package3d_urn="urn:adsk.eagle:package:15797/1"/>
 <part name="LED6" library="led" library_urn="urn:adsk.eagle:library:259" deviceset="LED" device="3MM" package3d_urn="urn:adsk.eagle:package:15797/1"/>
-<part name="VIN" library="adafruit" deviceset="1X2" device="-3.5MM"/>
 <part name="GPIO_DIG" library="pinhead" library_urn="urn:adsk.eagle:library:325" deviceset="PINHD-2X10" device="" package3d_urn="urn:adsk.eagle:package:22405/2"/>
 <part name="J1" library="adafruit" deviceset="1X2" device="-3.5MM"/>
@@
 <part name="SW_M2" library="pinhead" library_urn="urn:adsk.eagle:library:325" deviceset="PINHD-2X2" device="" package3d_urn="urn:adsk.eagle:package:22455/2"/>
 <part name="SW_M3" library="pinhead" library_urn="urn:adsk.eagle:library:325" deviceset="PINHD-2X2" device="" package3d_urn="urn:adsk.eagle:package:22455/2"/>
-<part name="J2" library="adafruit" deviceset="1X2" device="-3.5MM"/>
 <part name="J3" library="adafruit" deviceset="1X2" device="-3.5MM"/>
+<part name="Q1" library="transistor-npn" library_urn="urn:adsk.eagle:library:398" deviceset="BC817*" device="SMD" package3d_urn="urn:adsk.eagle:package:28748/2" technology="-25"/>
+<part name="U$1" library="RELAY" deviceset="RELAY" device=""/>
+<part name="D1" library="diode" library_urn="urn:adsk.eagle:library:210" deviceset="1N4004" device="" package3d_urn="urn:adsk.eagle:package:43336/1"/>
+<part name="VIN1" library="adafruit" deviceset="1X2" device="-3.5MM"/>
+<part name="R7" library="Resistor" deviceset="R" device="CHIP-0805(2012-METRIC)" package3d_urn="urn:adsk.eagle:package:16378559/2" technology="_"/>
 </parts>
 <sheets>
@@
 <attribute name="VALUE" x="10.795" y="61.468" size="1.778" layer="96" rot="R90"/>
 </instance>
-<instance part="VIN" gate="G$1" x="-40.64" y="194.31" smashed="yes" rot="R180"/>
 <instance part="GPIO_DIG" gate="A" x="180.34" y="86.36" smashed="yes">
 <attribute name="NAME" x="173.99" y="99.695" size="1.778" layer="95"/>
@@
 <attribute name="VALUE" x="242.57" y="71.12" size="1.778" layer="96"/>
 </instance>
-<instance part="J2" gate="G$1" x="-40.64" y="170.18" smashed="yes" rot="R180"/>
 <instance part="J3" gate="G$1" x="-40.64" y="181.61" smashed="yes" rot="R180"/>
+<instance part="Q1" gate="G$1" x="264.16" y="151.13" smashed="yes">
+<attribute name="NAME" x="267.97" y="149.86" size="1.778" layer="95"/>
+<attribute name="VALUE" x="267.97" y="147.32" size="1.778" layer="96"/>
+</instance>
+<instance part="U$1" gate="G$1" x="283.21" y="166.37" smashed="yes"/>
+<instance part="D1" gate="1" x="266.7" y="165.1" smashed="yes" rot="R90">
+<attribute name="NAME" x="266.2174" y="167.64" size="1.778" layer="95" rot="R90"/>
+<attribute name="VALUE" x="269.0114" y="167.64" size="1.778" layer="96" rot="R90"/>
+</instance>
+<instance part="VIN1" gate="G$1" x="308.61" y="165.1" smashed="yes"/>
+<instance part="R7" gate="G$1" x="255.27" y="151.13" smashed="yes" rot="R180">
+<attribute name="NAME" x="259.08" y="149.6314" size="1.778" layer="95" rot="R180"/>
+<attribute name="VALUE" x="259.08" y="154.432" size="1.778" layer="96" rot="R180"/>
+</instance>
 </instances>
 <busses>
@@
 <segment>
 <pinref part="J1" gate="G$1" pin="1"/>
+<label x="-30.48" y="167.64" size="1.27" layer="95" xref="yes"/>
 <wire x1="-35.56" y1="167.64" x2="-30.48" y2="167.64" width="0.1524" layer="91"/>
 <label x="-30.48" y="167.64" size="1.27" layer="95" xref="yes"/>
-<pinref part="J2" gate="G$1" pin="1"/>
-<wire x1="-35.56" y1="167.64" x2="-30.48" y2="167.64" width="0.1524" layer="91"/>
-<label x="-30.48" y="167.64" size="1.27" layer="95" xref="yes"/>
+<wire x1="-36.83" y1="167.64" x2="-35.56" y2="167.64" width="0.1524" layer="91"/>
 </segment>
 <segment>
@@
 </segment>
 <segment>
-<pinref part="VIN" gate="G$1" pin="1"/>
-<wire x1="-35.56" y1="191.77" x2="-30.48" y2="191.77" width="0.1524" layer="91"/>
-<label x="-30.48" y="191.77" size="1.016" layer="95" ratio="6" xref="yes"/>
+<pinref part="Q1" gate="G$1" pin="E"/>
+<wire x1="266.7" y1="146.05" x2="266.7" y2="133.35" width="0.1524" layer="91"/>
+<wire x1="266.7" y1="133.35" x2="243.84" y2="133.35" width="0.1524" layer="91"/>
+<label x="243.84" y="133.35" size="1.778" layer="95" rot="R180" xref="yes"/>
 </segment>
 </net>
@@
 </segment>
 <segment>
-<pinref part="VIN" gate="G$1" pin="2"/>
-<wire x1="-35.56" y1="194.31" x2="-30.48" y2="194.31" width="0.1524" layer="91"/>
-<label x="-30.48" y="194.31" size="1.016" layer="95" ratio="6" xref="yes"/>
+<pinref part="D1" gate="1" pin="C"/>
+<pinref part="U$1" gate="G$1" pin="IN"/>
+<wire x1="266.7" y1="167.64" x2="266.7" y2="173.99" width="0.1524" layer="91"/>
+<wire x1="266.7" y1="173.99" x2="278.13" y2="173.99" width="0.1524" layer="91"/>
+<wire x1="266.7" y1="173.99" x2="243.84" y2="173.99" width="0.1524" layer="91"/>
+<junction x="266.7" y="173.99"/>
+<label x="242.57" y="173.99" size="1.778" layer="95" rot="R180" xref="yes"/>
 </segment>
 </net>
@@
 </segment>
 <segment>
-<pinref part="J1" gate="G$1" pin="2"/>
+<label x="-30.48" y="170.18" size="1.27" layer="95" xref="yes"/>
 <wire x1="-35.56" y1="170.18" x2="-30.48" y2="170.18" width="0.1524" layer="91"/>
 <label x="-30.48" y="170.18" size="1.27" layer="95" xref="yes"/>
-<pinref part="J2" gate="G$1" pin="2"/>
-<wire x1="-35.56" y1="170.18" x2="-30.48" y2="170.18" width="0.1524" layer="91"/>
-<label x="-30.48" y="170.18" size="1.27" layer="95" xref="yes"/>
+<pinref part="J1" gate="G$1" pin="2"/>
 </segment>
 </net>
@@
 </segment>
 </net>
-<net name="LED_AUX" class="0">
-<segment>
-<pinref part="ARDUINOMEGA2560" gate="G$1" pin="11"/>
-<wire x1="135.89" y1="116.84" x2="147.32" y2="116.84" width="0.1524" layer="91"/>
-<label x="147.32" y="116.84" size="0.6096" layer="95" ratio="6" xref="yes"/>
-</segment>
-</net>
 <net name="FOCO_PIN" class="0">
 <segment>
@@
 <label x="123.19" y="39.37" size="0.6096" layer="95" rot="R270" xref="yes"/>
 </segment>
-</net>
+<segment>
+<pinref part="R7" gate="G$1" pin="2"/>
+<wire x1="250.19" y1="151.13" x2="243.84" y2="151.13" width="0.1524" layer="91"/>
+<label x="243.84" y="151.13" size="1.778" layer="95" rot="R180" xref="yes"/>
+</segment>
+</net>
+<net name="N$2" class="0">
+<segment>
+<pinref part="Q1" gate="G$1" pin="C"/>
+<pinref part="D1" gate="1" pin="A"/>
+<wire x1="266.7" y1="156.21" x2="266.7" y2="158.75" width="0.1524" layer="91"/>
+<pinref part="U$1" gate="G$1" pin="GND"/>
+<wire x1="266.7" y1="158.75" x2="266.7" y2="162.56" width="0.1524" layer="91"/>
+<wire x1="278.13" y1="158.75" x2="266.7" y2="158.75" width="0.1524" layer="91"/>
+<junction x="266.7" y="158.75"/>
+</segment>
+</net>
+<net name="N$1" class="0">
+<segment>
+<pinref part="U$1" gate="G$1" pin="COM-OPEN"/>
+<wire x1="285.75" y1="173.99" x2="303.53" y2="173.99" width="0.1524" layer="91"/>
+<pinref part="VIN1" gate="G$1" pin="1"/>
+<wire x1="303.53" y1="173.99" x2="303.53" y2="167.64" width="0.1524" layer="91"/>
+</segment>
+</net>
+<net name="N$3" class="0">
+<segment>
+<pinref part="U$1" gate="G$1" pin="COM-CLOSE"/>
+<wire x1="285.75" y1="158.75" x2="303.53" y2="158.75" width="0.1524" layer="91"/>
+<pinref part="VIN1" gate="G$1" pin="2"/>
+<wire x1="303.53" y1="158.75" x2="303.53" y2="165.1" width="0.1524" layer="91"/>
+</segment>
+</net>
+<net name="N$4" class="0">
+<segment>
+<pinref part="R7" gate="G$1" pin="1"/>
+<pinref part="Q1" gate="G$1" pin="B"/>
+<wire x1="260.35" y1="151.13" x2="261.62" y2="151.13" width="0.1524" layer="91"/>
+</segment>
+</net>

Commit message: PCB Corregidas
Parts:
- removed RELAYS: PINHD-1X4, Connector:PINHD-1X4
- R2, R3: device rcl:R-EU_0309/10 -> Resistor:R_CHIP-0805(2012-METRIC)
Connections:
- removed net D2: ARDUINOMEGA2560.2
- removed net D28: RELAYS.1
- removed net D29: RELAYS.2
- removed net D3: ARDUINOMEGA2560.3
- removed net D30: RELAYS.3
- removed net D4: ARDUINOMEGA2560.4
- removed net D5: ARDUINOMEGA2560.5
- removed net N$21: LED2.C, R2.2
- removed net N$22: LED3.C, R3.2
- new net N$5: LED2.A, R2.1
- new net N$6: LED3.A, R3.1
- net D31: now also ARDUINOMEGA2560.31; no longer RELAYS.4
- net D32: no longer ARDUINOMEGA2560.32
- net D33: no longer ARDUINOMEGA2560.33
- net D34: no longer ARDUINOMEGA2560.34
- net D35: no longer ARDUINOMEGA2560.35
- net D36: no longer ARDUINOMEGA2560.36
- net D37: no longer ARDUINOMEGA2560.37
- net D42: no longer ARDUINOMEGA2560.42
- net D43: no longer ARDUINOMEGA2560.43
- net D44: no longer ARDUINOMEGA2560.44
- net D45: no longer ARDUINOMEGA2560.45
- net D46: no longer ARDUINOMEGA2560.46
- net D47: no longer ARDUINOMEGA2560.47
- net D48: no longer ARDUINOMEGA2560.48
- net DIR_1: now also ARDUINOMEGA2560.30; no longer ARDUINOMEGA2560.23
- net DIR_2: now also ARDUINOMEGA2560.34; no longer ARDUINOMEGA2560.25
- net DIR_3: now also ARDUINOMEGA2560.37; no longer ARDUINOMEGA2560.27
- net FOCO_PIN: now also ARDUINOMEGA2560.48; no longer ARDUINOMEGA2560.31
- net GND: now also LED2.C, LED3.C; no longer R2.1, R3.1
- net LED_MOT_1: no longer ARDUINOMEGA2560.8
- net LED_MOT_2: now also ARDUINOMEGA2560.3; no longer ARDUINOMEGA2560.9
- net LED_MOT_3: now also ARDUINOMEGA2560.2; no longer ARDUINOMEGA2560.10
- net LED_SERV_1: now also ARDUINOMEGA2560.5, R2.2; no longer ARDUINOMEGA2560.7, LED2.A
- net LED_SERV_2: now also ARDUINOMEGA2560.11, R3.2; no longer ARDUINOMEGA2560.13, LED3.A
- net M2_ENABLE: now also ARDUINOMEGA2560.32; no longer ARDUINOMEGA2560.29
- net M3_ENABLE: now also ARDUINOMEGA2560.35; no longer ARDUINOMEGA2560.30
- net N$1: now also VIN1.2; no longer VIN1.1
- net N$3: now also U$1.COM, VIN1.1; no longer U$1.COM-CLOSE, VIN1.2
- net PWM_SERV_1: now also ARDUINOMEGA2560.4; no longer ARDUINOMEGA2560.6
- net PWM_SERV_2: now also ARDUINOMEGA2560.10; no longer ARDUINOMEGA2560.12
- net RX: now also UART_0.1; no longer UART_0.2
- net RX_3: now also UART_1.1; no longer UART_1.2
- net STEP_1: now also ARDUINOMEGA2560.29; no longer ARDUINOMEGA2560.22
- net STEP_2: now also ARDUINOMEGA2560.33; no longer ARDUINOMEGA2560.24
- net STEP_3: now also ARDUINOMEGA2560.36; no longer ARDUINOMEGA2560.26
- net TX: now also UART_0.2; no longer UART_0.1
- net TX_3: now also UART_1.2; no longer UART_1.1
Other:
- moved on the sheet: LED2, LED3, R2, R3

Commit message: Diseño PCB full
Parts:
- removed GPIO_DIG: (no value), pinhead:PINHD-2X10
- removed J1, J3, VIN1: 1X2-3.5MM, adafruit:1X2-3.5MM
- added JP1, JP2, JP3: (no value), adafruit:PINHD-2X4
- added R8: (no value), Resistor:R_CHIP-0805(2012-METRIC)
- added RESET: (no value), switch-omron:10-XX
- added X1, X2, X3: (no value), con-ptr500:AK300/2
Connections:
- removed net D32: GPIO_DIG.1
- removed net D33: GPIO_DIG.2
- removed net D34: GPIO_DIG.3
- removed net D35: GPIO_DIG.4
- removed net D36: GPIO_DIG.5
- removed net D37: GPIO_DIG.6
- removed net D48: GPIO_DIG.17
- new net D22: ARDUINOMEGA2560.22, JP3.4
- new net D23: ARDUINOMEGA2560.23, JP3.3
- new net D24: ARDUINOMEGA2560.24, JP3.6
- new net D25: ARDUINOMEGA2560.25, JP3.5
- new net D26: ARDUINOMEGA2560.26, JP3.8
- new net D27: ARDUINOMEGA2560.27, JP3.7
- new net RESET: ARDUINOMEGA2560.RESET, R8.2, RESET.P
- net D38: now also JP1.4; no longer GPIO_DIG.7
- net D39: now also JP1.3; no longer GPIO_DIG.8
- net D40: now also JP1.6; no longer GPIO_DIG.9
- net D41: now also JP1.5; no longer GPIO_DIG.10
- net D42: now also ARDUINOMEGA2560.42, JP1.8; no longer GPIO_DIG.11
- net D43: now also ARDUINOMEGA2560.43, JP1.7; no longer GPIO_DIG.12
- net D44: now also ARDUINOMEGA2560.44, JP2.2; no longer GPIO_DIG.13
- net D45: now also ARDUINOMEGA2560.45, JP2.1; no longer GPIO_DIG.14
- net D46: now also ARDUINOMEGA2560.46, JP2.4; no longer GPIO_DIG.15
- net D47: now also ARDUINOMEGA2560.47, JP2.3; no longer GPIO_DIG.16
- net D49: now also JP2.5; no longer GPIO_DIG.18
- net GND: now also JP1.1, JP1.2, JP2.6, JP2.7, JP2.8, RESET.S, X1-1.KL, X2-1.KL; no longer GPIO_DIG.19, GPIO_DIG.20, J1.1, J3.1
- net N$1: now also X3-2.KL; no longer VIN1.2
- net N$3: now also X3-1.KL; no longer VIN1.1
- net VCC_5: now also JP3.1, JP3.2, R8.1
- net VCC_MOT: now also X2-2.KL; no longer J1.2
- net VCC_SERVO: now also X1-2.KL; no longer J3.2

Commit message: Correcciones PCB
Parts:
- renumbered JP1 to DAUX_1, JP2 to DAUX2, JP3 to DAUX_3, LED1 to LED.ON, LED2 to LS_1, LED3 to LS_2, LED4 to LM_3, LED5 to LM_2, LED6 to LM_1, X1 to +6V, X2 to +12V, X3 to FOCO
Connections:
- net LED_MOT_1: now also ARDUINOMEGA2560.12
